Commit message: HoloMotion v1.4 sim teleop: reference-action replay pipeline, rot0 stereo robot, black hands, Isaac re-render
The teleop stack as used for the October rot0 recordings and their replays, merged onto the branch's packaged layout
(tasks in simple.tasks, generated MJCF in the scene cache, hbvcam bundle in src/simple/resources).

Replay
- simple.cli.rerecord_holomotion_v14 (new): closed-loop stored-input replay. Feeds the node the recorded reference frames,
  PICO sample and clock each 20 ms from the frame-0 snapshot; HoloMotion recomputes its outputs, physics re-runs; every
  frame's physics and model I/O are compared with the recording (bit-exact on the 50 rot0 episodes). Writes a new dataset
  (option --black-hands). --reference-source recorded | action | state | action_upper | state_upper swaps the joint channels
  of every reference frame for the model's own outputs or the measured joints (the 2026-10-19 experiment).
- simple.cli.replay_holomotion_v14: physics / action modes from the exact log, --video (head | third person), rebuilt robot
  with the recorded hand colour; _build_env fixed for tilt 0 + backpack.
- teleop/holomotion_v14/node_state.py (new): snapshot / restore / fresh_start of the node (reference queue, KV cache,
  yaw alignment, stick filter, evaluator caches) -> cold-start replay from frame 0. exact_log stores it (extra=).
- scripts/holomotion_v14_checks/: replay_node_from_dataset.py (open-loop node replay from the dataset columns),
  reference_actions_column_test.py (window column == rebuilt window; window-only replay bit-exact).
- docs/HOLOMOTION_V14_INPUT_REPLAY_HANDOFF.md: what the model needs, what the recording holds, how the replay feeds it.

Recording (teleop CLI)
- reference_actions (11 x 65 = 715) + reference_actions_frame_index: the node's window after each step (the v1.3 name),
  holomotion.tick_time, holomotion.* raw I/O, frame-0 node + agent snapshot; realformat columns derived live.
- --record-size 640x360 (both rectified eyes, intrinsics scaled in meta/holomotion_raw.json); --black-hands default on;
  resume guard (a dataset of another column set refuses to be appended to); skeleton cleanup; clean exit on errors.
- robot_variants: HBVCAM stereo head on the rot0 bracket (the 2026-10-16 base; legacy= rebuilds the rot15 September
  robot), both pinhole eyes, black Dex3 hands (visual only), generated XML in the scene cache (kerou's layout kept).

Eval / render
- eval_holomotion_v14: --black-hands, 640x360 per eye, both eyes sent under the recording's keys (merged with the
  fixed-eval-set handling of 1c33ca1).
- scripts/render_teleop_isaac.py: --eyes left,right, --seed (one look), --look-from <episodes.jsonl> (the same-background
  materials + lights, --look-light-scale), --out-size; scripts/install_isaac_renders.py installs the renders as a
  dataset's ego-view videos. isaac_views.PinholeCamera(eye).
- hbvcam bundle: rot0 base files + the rot15 ones kept, SOURCE.md.

Packaged tasks: <KIT>_ROBOT=g1 (set by the HoloMotion loader) keeps SIMPLE's stock G1Sonic with the teleop MJCF; the default
(g1comp) is unchanged for the evaluations. Verified from this branch's source: rerecord episode 0 of the rot0 set -> physics
and policy I/O bit-exact, task success; replay_holomotion_v14 --mode physics bit-exact (the saved-model hash differs because
the generated MJCF now lives in the scene cache with absolute mesh paths; mj_saveModel hashes include path strings).

Not in the repo: model_22000 (NAS-28, see docs/holomotion_v14_teleop.md), the recordings, the generated runbook HTML
(ignored on this branch; NAS http://10.40.11.11:8899/pico_sim_teleop_runbook.html).

Co-Authored-By: Claude Fable 5.1 <noreply@anthropic.com>

File: src/simple/resources/hbvcam_stereo/g1_29dof_with_hand_hbvcam_stereo.urdf (robot description, URDF)
Before this commit: robot g1_29dof_with_hand_hbvcam_stereo, 56 links, 55 joints
Joints:
- joint head_stereo_joint: origin xyz=0.0677735505 0 0.4264672285 rpy=0 0.598492592 0 -> xyz=0.070323550 0.000000000 0.424707229 rpy=0.000000000 0.860291980 0.000000000
- joint head_stereo_left_optical_joint: origin xyz=0.067974825 0.030355827 0.426216236 rpy=-2.169288919 0.000000000 -1.570796327 -> xyz=0.070524825 0.030355827 0.424456236 rpy=-2.431088307 0.000000000 -1.570796327
- joint head_stereo_right_optical_joint: origin xyz=0.067572276 -0.030355827 0.426718221 rpy=-2.169646752 -0.002785440 -1.576804238 -> xyz=0.070122276 -0.030355827 0.424958221 rpy=-2.431446140 -0.002785440 -1.576804238
